File: wheel_robot_kicad/wheel_robot_kicad.kicad_sch (KiCad schematic)
At the start: 8 parts, among them U4 Mini360, U6 TB6612FNG, U8 ESP32-S3-DEVKITC-1-N8R8

Commit message: added pull up resistors
Parts:
- added R3, R4: 6.8k, symbol Device:R
Connections:
- net at U7.2 (3v3), U7.6 (CS), U8.J1_1 (3V3): now also R3.1, R4.1
- net at U7.4 (SCL), U8.J3_12 (GPIO36): now also R3.2
- net at U7.5 (SDA), U8.J3_13 (GPIO35): now also R4.2
Changed lines of the file:
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@@
+	)
+	(junction
+		(at 38.1 93.98)
+		(diameter 0)
+		(color 0 0 0 0)
 	)
 	(junction
@@
 	)
 	(junction
+		(at 36.83 91.44)
+		(diameter 0)
+		(color 0 0 0 0)
+	)
+	(junction
 		(at 148.59 114.3)
 		(diameter 0)
@@
 	)
 	(junction
+		(at 26.67 83.82)
+		(diameter 0)
+		(color 0 0 0 0)
+	)
+	(junction
 		(at 87.63 99.06)
 		(diameter 0)
@@
 	(wire
 		(pts
-			(xy 182.88 71.12) (xy 179.07 71.12)
+			(xy 189.23 71.12) (xy 179.07 71.12)
 		)
 		(stroke
@@
 	(wire
 		(pts
+			(xy 26.67 91.44) (xy 36.83 91.44)
+		)
+		(stroke
+			(width 0)
+			(type default)
+		)
+	)
+	(wire
+		(pts
 			(xy 34.29 156.21) (xy 34.29 83.82)
 		)
@@
 	(wire
 		(pts
+			(xy 38.1 93.98) (xy 38.1 121.92)
+		)
+		(stroke
+			(width 0)
+			(type default)
+		)
+	)
+	(wire
+		(pts
 			(xy 92.71 87.63) (xy 92.71 137.16)
 		)
@@
 	(wire
 		(pts
+			(xy 36.83 91.44) (xy 36.83 124.46)
+		)
+		(stroke
+			(width 0)
+			(type default)
+		)
+	)
+	(wire
+		(pts
 			(xy 91.44 139.7) (xy 86.36 139.7)
 		)
@@
 	(wire
 		(pts
-			(xy 36.83 78.74) (xy 36.83 124.46)
+			(xy 36.83 78.74) (xy 36.83 91.44)
 		)
 		(stroke
@@
 	(wire
 		(pts
+			(xy 26.67 83.82) (xy 34.29 83.82)
+		)
+		(stroke
+			(width 0)
+			(type default)
+		)
+	)
+	(wire
+		(pts
 			(xy 158.75 135.89) (xy 168.91 135.89)
 		)
@@
 	(wire
 		(pts
-			(xy 182.88 121.92) (xy 176.53 121.92)
+			(xy 189.23 121.92) (xy 176.53 121.92)
 		)
 		(stroke
@@
 	(wire
 		(pts
+			(xy 17.78 91.44) (xy 17.78 93.98)
+		)
+		(stroke
+			(width 0)
+			(type default)
+		)
+	)
+	(wire
+		(pts
 			(xy 86.36 152.4) (xy 86.36 156.21)
 		)
@@
 	(wire
 		(pts
-			(xy 182.88 71.12) (xy 182.88 121.92)
+			(xy 189.23 71.12) (xy 189.23 121.92)
 		)
 		(stroke
@@
 	(wire
 		(pts
-			(xy 38.1 81.28) (xy 38.1 121.92)
+			(xy 38.1 81.28) (xy 38.1 93.98)
 		)
 		(stroke
@@
 	(wire
 		(pts
+			(xy 17.78 93.98) (xy 38.1 93.98)
+		)
+		(stroke
+			(width 0)
+			(type default)
+		)
+	)
+	(wire
+		(pts
 			(xy 148.59 76.2) (xy 148.59 99.06)
+		)
+		(stroke
+			(width 0)
+			(type default)
+		)
+	)
+	(wire
+		(pts
+			(xy 17.78 83.82) (xy 26.67 83.82)
 		)
 		(stroke
@@
 	)
 	(symbol
+		(lib_id "Device:R")
+		(at 26.67 87.63 0)
+		(unit 1)
+		(exclude_from_sim no)
+		(in_bom yes)
+		(on_board yes)
+		(dnp no)
+		(fields_autoplaced yes)
+		(property "Reference" "R3"
+			(at 29.21 86.3599 0)
+			(effects
+				(font
+					(size 1.27 1.27)
+				)
+				(justify left)
+			)
+		)
+		(property "Value" "6.8k"
+			(at 29.21 88.8999 0)
+			(effects
+				(font
+					(size 1.27 1.27)
+				)
+				(justify left)
+			)
+		)
+		(property "Footprint" ""
+			(at 24.892 87.63 90)
+			(effects
+				(font
+					(size 1.27 1.27)
+				)
+				(hide yes)
+			)
+		)
+		(property "Datasheet" "~"
+			(at 26.67 87.63 0)
+			(effects
+				(font
+					(size 1.27 1.27)
+				)
+				(hide yes)
+			)
+		)
+		(property "Description" "Resistor"
+			(at 26.67 87.63 0)
+			(effects
+				(font
+					(size 1.27 1.27)
+				)
+				(hide yes)
+			)
+		)
+		(pin "2"
+		)
+		(pin "1"
+		)
+		(instances
+			(project ""
+				(path "/228a0b42-286a-4357-814d-e937725b6893"
+					(reference "R3")
+					(unit 1)
+				)
+			)
+		)
+	)
+	(symbol
 		(lib_id "Driver_Motor:TB6612FNG")
 		(at 123.19 106.68 270)
@@
 					(unit 1)
 				)
+			)
+		)
+	)
+	(symbol
+		(lib_id "Device:R")
+		(at 17.78 87.63 0)
+		(unit 1)
+		(exclude_from_sim no)
+		(in_bom yes)
+		(on_board yes)
+		(dnp no)
+		(fields_autoplaced yes)
+		(property "Reference" "R4"
+			(at 20.32 86.3599 0)
+			(effects
+				(font
+					(size 1.27 1.27)
+				)
+				(justify left)
+			)
+		)
+		(property "Value" "6.8k"
+			(at 20.32 88.8999 0)
+			(effects
+				(font
+					(size 1.27 1.27)
+				)
+				(justify left)
+			)
+		)
+		(property "Footprint" ""
+			(at 16.002 87.63 90)
+			(effects
+				(font
+					(size 1.27 1.27)
+				)
+				(hide yes)
+			)
+		)
+		(property "Datasheet" "~"
+			(at 17.78 87.63 0)
+			(effects
+				(font
+					(size 1.27 1.27)
+				)
+				(hide yes)
+			)
+		)
+		(property "Description" "Resistor"
+			(at 17.78 87.63 0)
+			(effects
+				(font
+					(size 1.27 1.27)
+				)
+				(hide yes)
+			)
+		)
+		(pin "2"
+		)
+		(pin "1"
+		)
+		(instances
+			(project ""
+				(path "/228a0b42-286a-4357-814d-e937725b6893"
+					(reference "R4")
+					(unit 1)
+				)
